File: SerialHub.kicad_pcb (KiCad board)
At the start: 4 copper layers, 90.7 x 78.1 mm, 127 parts, among them J1 Conn_01x04_Pin, J10 USB_C_Receptacle_USB2.0_16P, J11 Conn_01x04_Pin, J12 USB_C_Receptacle_USB2.0_16P, J15 Conn_02x24_Odd_Even, J2 USB_C_Receptacle_USB2.0_16P, J3 Conn_01x04_Pin, J4 USB_C_Receptacle_USB2.0_16P, J5 Conn_01x04_Pin, J6 USB_C_Receptacle_USB2.0_16P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

Commit message: Order
Parts:
- added C69: 100nF, Capacitor_SMD:C_0402_1005Metric, F.Cu at (180.8, 118.6)
- added C70: 100nF, Capacitor_SMD:C_0402_1005Metric, F.Cu at (168.8, 79.2)
- R11, R12, R15, R16, R19, R20, R23, R24, R3, R4, R7, R8: value 27.4Ω -> 27Ω
- R27, R28, R29, R30, R31: value 7.5kΩ -> 7.15kΩ
- SW1: footprint Button_Switch_SMD:SW_SPST_PTS647_Sx38 -> Button_Switch_THT:SW_PUSH_6mm_H4.3mm
- moved SW1 34.3 mm to (162.3, 83.1)
- moved G*** 32.7 mm to (152.2, 102.6)
- moved C1 32.6 mm to (185.9, 94.5)
- moved C13 32.6 mm to (183.7, 88.0)
- moved C16 32.6 mm to (183.7, 107.2)
- moved C24 32.6 mm to (183.7, 108.2)
- moved C25 32.6 mm to (162.6, 128.8)
- moved C32 32.6 mm to (166.6, 126.2)
- moved C33 32.6 mm to (155.8, 126.2)
- moved C37 32.6 mm to (140.4, 116.3)
- moved C41 32.6 mm to (141.4, 128.4)
- moved C42 32.6 mm to (141.4, 116.3)
- moved C45 32.6 mm to (135.2, 121.2)
- moved C5 32.6 mm to (183.7, 87.0)
- moved C59 32.6 mm to (130.2, 85.1)
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Routing:
- net /MCU/RUN: track 18.7 -> 26.9 mm
- net GND: vias 120 -> 118
Other:
- board size 90.7 x 78.1 mm -> 90.7 x 78.2 mm
