File: SerialHub.kicad_sch (KiCad schematic)
At the start: 18 parts, among them J15 Conn_02x24_Odd_Even, SW1 SW_SPST, U2 W25Q16JVSS, U9 TLV74033PDBVR, X1 ASE-12.000MHz-E-T

Commit message: Added Schematic PDF
Parts:
- H1, H2, H3, H4: footprint (none) -> MountingHole:MountingHole_3.2mm_M3_Pad
Changed lines of the file:
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@@
 			)
 		)
-		(property "Footprint" ""
+		(property "Footprint" "MountingHole:MountingHole_3.2mm_M3_Pad"
 			(at 241.3 161.29 0)
 			(effects
@@
 			)
 		)
-		(property "Footprint" ""
+		(property "Footprint" "MountingHole:MountingHole_3.2mm_M3_Pad"
 			(at 247.65 161.29 0)
 			(effects
@@
 			)
 		)
-		(property "Footprint" ""
+		(property "Footprint" "MountingHole:MountingHole_3.2mm_M3_Pad"
 			(at 260.35 161.29 0)
 			(effects
@@
 			)
 		)
-		(property "Footprint" ""
+		(property "Footprint" "MountingHole:MountingHole_3.2mm_M3_Pad"
 			(at 254 161.29 0)
 			(effects

Commit message: Order
Parts:
- added C69, C70: 100nF, Capacitor_SMD:C_0402_1005Metric, symbol Device:C
- C1, C2: Digikey (none) -> 399-C0402C105K9PACTUCT-ND
- J15: now left out of the parts list
- R1, R2: Digikey (none) -> 311-10KJRCT-ND
- R27, R28, R29, R30, R31: value 7.5kΩ -> 7.15kΩ; Digikey (none) -> YAG3235CT-ND
- SW1: footprint Button_Switch_SMD:SW_SPST_PTS647_Sx38 -> Button_Switch_THT:SW_PUSH_6mm_H4.3mm; Digikey (none) -> 2223-TS02-66-43-BK-160-LCR-D-ND
- U2: Digikey (none) -> 256-W25Q16JVSSIQTRCT-ND
- U9: Digikey (none) -> 296-TLV74033PDBVRCT-ND
- X1: Digikey (none) -> 535-ASE-12.000MHZ-E-TCT-ND
Connections:
- net +3.3V: now also C69.1, C70.1
- net GND: now also C69.2, C70.2
