File: untitled.kicad_sch (KiCad schematic)
At the start: 18 parts, among them J1 Conn_01x04_Pin, J2 USB_C_Receptacle_USB2.0_16P, U3 RP2040

Commit message: Added Schematic PDF
Changed lines of the file:
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@@
 	(generator "eeschema")
 	(generator_version "9.0")
-	(paper "A4")
+	(paper "USLetter")
 	(text "1uF near VREG_IN\n1uF near VREG_VOUT"
 		(exclude_from_sim no)
@@
 					(size 1.27 1.27)
 				)
+				(hide yes)
 			)
 		)
@@
 		(on_board yes)
 		(dnp no)
-		(fields_autoplaced yes)
 		(property "Reference" "R4"
-			(at 41.275 52.07 0)
+			(at 35.814 56.134 90)
 			(effects
 				(font
@@
 		)
 		(property "Value" "27.4Ω"
-			(at 41.275 54.61 0)
+			(at 37.338 56.134 90)
 			(effects
 				(font
@@
 		(on_board yes)
 		(dnp no)
-		(fields_autoplaced yes)
 		(property "Reference" "R5"
-			(at 47.625 52.07 0)
+			(at 42.164 56.134 90)
 			(effects
 				(font
@@
 		)
 		(property "Value" "5.11kΩ"
-			(at 47.625 54.61 0)
+			(at 43.688 56.134 90)
 			(effects
 				(font
@@
 		(on_board yes)
 		(dnp no)
-		(fields_autoplaced yes)
 		(property "Reference" "R6"
-			(at 53.975 52.07 0)
+			(at 48.514 56.134 90)
 			(effects
 				(font
@@
 		)
 		(property "Value" "5.11kΩ"
-			(at 53.975 54.61 0)
+			(at 50.038 56.134 90)
 			(effects
 				(font
@@
 		(on_board yes)
 		(dnp no)
-		(fields_autoplaced yes)
 		(property "Reference" "R3"
-			(at 34.925 52.07 0)
+			(at 29.464 56.134 90)
 			(effects
 				(font
@@
 		)
 		(property "Value" "27.4Ω"
-			(at 34.925 54.61 0)
+			(at 30.988 56.134 90)
 			(effects
 				(font

Commit message: Order
Parts:
- C10, C11, C12, C3, C4, C6, C7, C8, C9: Digikey (none) -> 1276-1043-1-ND
- C13, C5: Digikey (none) -> 399-C0402C105K9PACTUCT-ND
- J1: now left out of the parts list
- J2: Digikey (none) -> 2223-UJ20-C-H-G-SMT-1-P16-TRCT-ND
- R3, R4: value 27.4Ω -> 27Ω; Digikey (none) -> YAG5278CT-ND
- R5, R6: Digikey (none) -> RMCF0402FT5K11CT-ND
- U3: Digikey (none) -> 2648-SC0914(13)CT-ND
Changed lines of the file:
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@@
 		(unit 1)
 		(exclude_from_sim no)
-		(in_bom yes)
+		(in_bom no)
 		(on_board yes)
 		(dnp no)
@@
 			)
 		)
+		(property "Digikey" ""
+			(at 24.13 137.16 0)
+			(effects
+				(font
+					(size 1.27 1.27)
+				)
+				(hide yes)
+			)
+		)
 		(pin "3"
 		)
@@
 			)
 		)
+		(property "Digikey" "1276-1043-1-ND"
+			(at 67.945 36.195 90)
+			(effects
+				(font
+					(size 1.27 1.27)
+				)
+				(hide yes)
+			)
+		)
 		(pin "1"
 		)
@@
 			)
 		)
+		(property "Digikey" "2223-UJ20-C-H-G-SMT-1-P16-TRCT-ND"
+			(at 38.1 31.75 90)
+			(effects
+				(font
+					(size 1.27 1.27)
+				)
+				(hide yes)
+			)
+		)
 		(pin "A5"
 		)
@@
 					(size 1.27 1.27)
 				)
+			)
+		)
+		(property "Digikey" "1276-1043-1-ND"
+			(at 95.885 29.21 90)
+			(effects
+				(font
+					(size 1.27 1.27)
+				)
+				(hide yes)
 			)
 		)
@@
 			)
 		)
-		(property "Value" "27.4Ω"
+		(property "Value" "27Ω"
 			(at 37.338 56.134 90)
 			(effects
@@
 			)
 		)
+		(property "Digikey" "YAG5278CT-ND"
+			(at 39.37 53.34 90)
+			(effects
+				(font
+					(size 1.27 1.27)
+				)
+				(hide yes)
+			)
+		)
 		(pin "1"
 		)
@@
 			)
 		)
+		(property "Digikey" "1276-1043-1-ND"
+			(at 81.915 29.21 90)
+			(effects
+				(font
+					(size 1.27 1.27)
+				)
+				(hide yes)
+			)
+		)
 		(pin "1"
 		)
@@
 			)
 		)
+		(property "Digikey" "399-C0402C105K9PACTUCT-ND"
+			(at 67.945 43.18 90)
+			(effects
+				(font
+					(size 1.27 1.27)
+				)
+				(hide yes)
+			)
+		)
 		(pin "1"
 		)
@@
 			)
 		)
+		(property "Digikey" "RMCF0402FT5K11CT-ND"
+			(at 45.72 53.34 90)
+			(effects
+				(font
+					(size 1.27 1.27)
+				)
+				(hide yes)
+			)
+		)
 		(pin "1"
 		)
@@
 			)
 		)
+		(property "Digikey" "RMCF0402FT5K11CT-ND"
+			(at 52.07 53.34 90)
+			(effects
+				(font
+					(size 1.27 1.27)
+				)
+				(hide yes)
+			)
+		)
 		(pin "1"
 		)
@@
 					(size 1.27 1.27)
 				)
+			)
+		)
+		(property "Digikey" "1276-1043-1-ND"
+			(at 95.885 43.18 90)
+			(effects
+				(font
+					(size 1.27 1.27)
+				)
+				(hide yes)
 			)
 		)
@@
 			)
 		)
+		(property "Digikey" "1276-1043-1-ND"
+			(at 81.915 50.165 90)
+			(effects
+				(font
+					(size 1.27 1.27)
+				)
+				(hide yes)
+			)
+		)
 		(pin "1"
 		)
@@
 			)
 		)
+		(property "Digikey" "1276-1043-1-ND"
+			(at 95.885 36.195 90)
+			(effects
+				(font
+					(size 1.27 1.27)
+				)
+				(hide yes)
+			)
+		)
 		(pin "1"
 		)
@@
 			)
 		)
+		(property "Digikey" "2648-SC0914(13)CT-ND"
+			(at 66.04 106.68 0)
+			(effects
+				(font
+					(size 1.27 1.27)
+				)
+				(hide yes)
+			)
+		)
 		(pin "22"
 		)
@@
 			)
 		)
+		(property "Digikey" "1276-1043-1-ND"
+			(at 67.945 29.21 90)
+			(effects
+				(font
+					(size 1.27 1.27)
+				)
+				(hide yes)
+			)
+		)
 		(pin "1"
 		)
@@
 			)
 		)
+		(property "Digikey" "399-C0402C105K9PACTUCT-ND"
+			(at 95.885 50.165 90)
+			(effects
+				(font
+					(size 1.27 1.27)
+				)
+				(hide yes)
+			)
+		)
 		(pin "1"
 		)
@@
 			)
 		)
+		(property "Digikey" "1276-1043-1-ND"
+			(at 81.915 43.18 90)
+			(effects
+				(font
+					(size 1.27 1.27)
+				)
+				(hide yes)
+			)
+		)
 		(pin "1"
 		)
@@
 			)
 		)
-		(property "Value" "27.4Ω"
+		(property "Value" "27Ω"
 			(at 30.988 56.134 90)
 			(effects
@@
 			)
 		)
+		(property "Digikey" "YAG5278CT-ND"
+			(at 33.02 53.34 90)
+			(effects
+				(font
+					(size 1.27 1.27)
+				)
+				(hide yes)
+			)
+		)
 		(pin "1"
 		)
@@
 			)
 		)
+		(property "Digikey" "1276-1043-1-ND"
+			(at 81.915 36.195 90)
+			(effects
+				(font
+					(size 1.27 1.27)
+				)
+				(hide yes)
+			)
+		)
